File: power_supply.kicad_sch (KiCad schematic)
At the start: 28 parts, among them J2 USB_C_Receptacle_USB2.0_16P, J3 Battery, U2 AP2112K-3.3, U3 BQ25606RGER, U4 INA219AxD

Commit message: Working
Other:
- moved on the sheet: C21
