File: tinyPaper.kicad_pcb (KiCad board)
At the start: 4 copper layers, 80 x 60 mm, 69 parts, among them J1 ePaper Display, J2 USB_C_Receptacle_USB2.0_16P, J3 Battery, J4 External antenna, SW1 Boot, SW2 Reset, SW3 Boot, SW4 Boot, SW5 Boot, U1 ESP32-S3, U2 AP2112K-3.3, U3 BQ25606RGER, U4 INA219AxD, Y1 Crystal_GND24

Commit message: Working
Parts:
- moved R23 33.9 mm to (107.8, 121.0), turned to 0 degrees
- moved R22 33.1 mm to (141.2, 120.3), turned to 0 degrees
- moved SW4 32.8 mm to (73.2, 124.2)
- moved SW3 32.8 mm to (106.0, 124.5)
- moved C3 5.31 mm to (88.9, 115.3)
- moved U4 5.31 mm to (93.5, 116.4)
- moved R3 5.31 mm to (93.5, 111.5)
- moved R8 2.50 mm to (106.7, 102.7), turned to 90 degrees
- moved R7 2.50 mm to (104.2, 102.6)
- moved C14 1.81 mm to (115.3, 99.5)
- moved C13 1.81 mm to (115.3, 97.9)
- moved R2 1.60 mm to (134.7, 113.0), turned to 180 degrees
- moved R1 1.38 mm to (134.4, 110.1), turned to 180 degrees
- moved R21 0.39 mm to (75.0, 120.6)
- moved C2 0.28 mm to (101.1, 116.0)
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Connections:
- net /DISPLAY_BLK renamed DISPLAY_BLK
- net /DISPLAY_CS renamed DISPLAY_CS
- net /DISPLAY_DC renamed DISPLAY_DC
- net /DISPLAY_RST renamed DISPLAY_RST
- net /DISPLAY_SCK renamed DISPLAY_SCK
- net /DISPLAY_SDA renamed DISPLAY_SDA
- net /ESP_LNA renamed ESP_LNA
- net /Power supply/PMIC_USB_D+ renamed PMIC_USB_D+
- net /Power supply/PMIC_USB_D- renamed PMIC_USB_D-
- net /WIFI_ANTENNA renamed /WiFi/WIFI_ANTENNA
- net /WIFI_ANTENNA_EXT renamed /WiFi/WIFI_ANTENNA_EXT
- net /WIFI_ANTENNA_F renamed /WiFi/WIFI_ANTENNA_F
- net /WIFI_ANTENNA_PCB renamed /WiFi/WIFI_ANTENNA_PCB
- C11 pad 1: +3V3 -> 3V3
- C12 pad 1: +3V3 -> 3V3
- C15 pad 1: +3V3 -> 3V3
- C5 pad 1: +3V3 -> 3V3
- C7 pad 1: +3V3 -> 3V3
- C8 pad 1: +3V3 -> 3V3
- C9 pad 1: +3V3 -> 3V3
- J2 pad A6: /Power supply/USB_D+ -> USB_D+
- J2 pad A7: /Power supply/USB_D- -> USB_D-
- J2 pad B6: /Power supply/USB_D+ -> USB_D+
- J2 pad B7: /Power supply/USB_D- -> USB_D-
- L2 pad 1: +3V3 -> 3V3
- R11 pad 2: +3V3 -> 3V3
- R21 pad 1: +3V3 -> 3V3
- R22 pad 1: +3V3 -> 3V3
- R23 pad 1: +3V3 -> 3V3
- R6 pad 2: +3V3 -> 3V3
- R7 pad 1: METER_SDA -> METER_SCL
- R7 pad 2: +3V3 -> 3V3
- R8 pad 1: METER_SCL -> 3V3
- R8 pad 2: +3V3 -> METER_SDA
- SW3 pad 1: Net-(R21-Pad2) -> Net-(R23-Pad2)
- SW4 pad 1: Net-(R22-Pad2) -> Net-(R21-Pad2)
- SW5 pad 1: Net-(R23-Pad2) -> Net-(R22-Pad2)
- U1 pad 20: +3V3 -> 3V3
- U1 pad 25: /USB_D- -> USB_D-
- U1 pad 26: /USB_D+ -> USB_D+
- U1 pad 46: +3V3 -> 3V3
- U1 pad 55: +3V3 -> 3V3
- U1 pad 56: +3V3 -> 3V3
Routing:
- net Net-(U1-GPIO9): track 4.54 -> 73.8 mm, vias 1 -> 2
- net Net-(U1-GPIO8): track 6.20 -> 49.5 mm, vias 1 -> 2
- net USB_D+: track 0.00 -> 37.9 mm, vias 0 -> 2
- net VSYS: track 4.91 -> 42.4 mm, vias 0 -> 3
- net USB_D-: track 0.00 -> 36.9 mm, vias 0 -> 2
- net Net-(U1-GPIO7): track 7.63 -> 43.4 mm, vias 1 -> 2
- net /ESP_EN: track 79.9 -> 45.4 mm, vias 0 -> 2
- net /ESP_IO0: track 82.9 -> 48.8 mm, vias 0 -> 2
- net GND: track 0.00 -> 31.4 mm, vias 0 -> 21
- net 3V3: track 2.17 -> 31.9 mm, vias 0 -> 12
- net VBUS: track 0.00 -> 22.4 mm, vias 0 -> 2
- net VBAT: track 11.7 -> 32.7 mm
- net +3V3: track 17.7 -> 0.00 mm, vias 7 -> 0
- net DISPLAY_BLK: track 16.1 -> 2.05 mm, vias 2 -> 1
- net DISPLAY_DC: track 16.1 -> 2.83 mm, vias 2 -> 1
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- added copper zone on B.Cu, net 3V3
- added copper zone on In2.Cu, net GND
- added copper zone on F.Cu, net VBAT
- added copper zone on F.Cu, net VBUS
- added copper zone on F.Cu, net VSYS
- removed copper zone on B.Cu, net GND
