File: tinyPaper.kicad_sch (KiCad schematic)
At the start: 40 parts, among them J4 External antenna, SW1 Boot, SW2 Reset, SW3 Boot, SW4 Boot, SW5 Boot, U1 ESP32-S3, Y1 Crystal_GND24

Commit message: Working
Parts:
- removed AE1: PCB antenna, Library:ESPRESSIF_ESP32_MIFA_2.4GHz_Right, symbol Device:Antenna_Loop
- removed C16, C18, C19: LNA, Capacitor_SMD:C_0603_1608Metric, symbol Device:C
- removed J4: External antenna, Connector_Coaxial:U.FL_Hirose_U.FL-R-SMT-1_Vertical, symbol Connector:Conn_Coaxial
- removed L3, L4: L, Inductor_SMD:L_0603_1608Metric, symbol Device:L
- removed R12, R13: 0R, Resistor_SMD:R_0603_1608Metric, symbol Device:R
Connections:
- net METER_SCL: now also R7.1; no longer R8.1
- net METER_SDA: now also R8.2; no longer R7.1
- net at R22.2: now also SW5.1; no longer SW4.1
- net at R21.2: now also SW4.1; no longer SW3.1
- net at R23.2: now also SW3.1; no longer SW5.1
- net +3V3 renamed 3V3
- net 3V3: now also R8.1; no longer R8.2
Other:
- added sheet WiFi (wifi.kicad_sch)
- moved on the sheet: C10, C11, C12, C13, C14, C15, C17, C4, C5, C6, C7, C8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
